Commit message: Refactor Mecarosmaster launch and configuration files
- Updated `mecarosmaster_launch.py` to fix YAML parsing issue for `robot_description` by wrapping it in `ParameterValue`.
- Removed deprecated `mecarosmaster_controllers.yaml` file as its parameters are now integrated directly into the launch file.
- Enhanced the launch sequence to ensure proper initialization order of nodes and added delays for spawners to avoid race conditions.
- Modified `mecarosmaster_node.cpp` to correct joint names to match URDF definitions and improved the publish logic for joint states.
- Revamped `mecarosmaster.urdf.xacro` to include missing `ros2_control` block and ensure joint names align with the hardware plugin requirements.

File: mecarosmaster_ws/src/mecarosmaster_control/urdf/mecarosmaster.urdf.xacro (robot description, xacro)
@@ -1,73 +1,249 @@
-<?xml version="1.0"?>
-<robot name="mecarosmaster" xmlns:xacro="http://www.ros.org/wiki/xacro">
-  <xacro:arg name="serial_port" default="/dev/myserial" />
-  <xacro:arg name="car_type" default="1" />
+<?xml version="1.0" encoding="utf-8"?>
+<!--
+    mecarosmaster.urdf.xacro  —  ROS 2 Humble
+    Corrections :
+      • Noms de joints SANS préfixe namespace (front_left_joint, etc.)
+        pour correspondre au YAML et au hardware plugin.
+      • Bloc <ros2_control> ajouté (était totalement absent).
+      • Arguments xacro serial_port / car_type transmis au plugin.
+    Auteur : dirennoukpo <diren.noukpo@epitech.eu>
+-->
+<robot name="yahboomcar" xmlns:xacro="http://wiki.ros.org/xacro">
+  <!-- ── Arguments passés par le launch ──────────────────────────────────── -->
+  <xacro:arg name="serial_port" default="/dev/myserial"/>
+  <xacro:arg name="car_type"    default="1"/>
+  <!-- ── Matériaux ──────────────────────────────────────────────────────── -->
+  <material name="Green"><color rgba="0 0.7 0 1"/></material>
+  <material name="White"><color rgba="0.7 0.7 0.7 1"/></material>
+  <!-- ═══════════════════════════════════════════════════════════════════════
+       LIENS
+  ══════════════════════════════════════════════════════════════════════════ -->
+  <link name="base_footprint"/>
+  <link name="imu_link"/>
   <link name="base_link">
-    <visual>
-      <geometry>
-        <box size="0.32 0.28 0.08" />
-      </geometry>
-      <material name="gray">
-        <color rgba="0.6 0.6 0.6 1.0" />
-      </material>
-    </visual>
-    <collision>
-      <geometry>
-        <box size="0.32 0.28 0.08" />
-      </geometry>
-    </collision>
-  </link>
-  <link name="wheel_fl">
-    <visual>
-      <geometry>
-        <cylinder radius="0.045" length="0.02" />
-      </geometry>
-    </visual>
-  </link>
-  <link name="wheel_fr">
-    <visual>
-      <geometry>
-        <cylinder radius="0.045" length="0.02" />
-      </geometry>
-    </visual>
-  </link>
-  <link name="wheel_rl">
-    <visual>
-      <geometry>
-        <cylinder radius="0.045" length="0.02" />
-      </geometry>
-    </visual>
-  </link>
-  <link name="wheel_rr">
-    <visual>
-      <geometry>
-        <cylinder radius="0.045" length="0.02" />
-      </geometry>
-    </visual>
-  </link>
-  <joint name="wheel_fl_joint" type="continuous">
-    <parent link="base_link" />
-    <child link="wheel_fl" />
-    <origin xyz="0.14 0.12 0.0" rpy="0 1.5708 0" />
-    <axis xyz="0 0 1" />
-  </joint>
-  <joint name="wheel_fr_joint" type="continuous">
-    <parent link="base_link" />
-    <child link="wheel_fr" />
-    <origin xyz="0.14 -0.12 0.0" rpy="0 1.5708 0" />
-    <axis xyz="0 0 1" />
-  </joint>
-  <joint name="wheel_rl_joint" type="continuous">
-    <parent link="base_link" />
-    <child link="wheel_rl" />
-    <origin xyz="-0.14 0.12 0.0" rpy="0 1.5708 0" />
-    <axis xyz="0 0 1" />
-  </joint>
-  <joint name="wheel_rr_joint" type="continuous">
-    <parent link="base_link" />
-    <child link="wheel_rr" />
-    <origin xyz="-0.14 -0.12 0.0" rpy="0 1.5708 0" />
-    <axis xyz="0 0 1" />
-  </joint>
-  <xacro:include filename="$(find mecarosmaster_control)/urdf/ros2_control.xacro" />
+    <inertial>
+      <origin xyz="0.00498197982182523 5.70233829969297E-05 -0.0121008098068578" rpy="0 0 0"/>
+      <mass value="0.486218814966626"/>
+      <inertia ixx="0.00196277727666921" ixy="2.50447049446755E-07" ixz="0.000140534767811098"
+               iyy="0.00457256033711368" iyz="2.68618064993882E-07"  izz="0.00493927269870476"/>
+    </inertial>
+    <visual>
+      <origin xyz="0 0 0" rpy="0 0 0"/>
+      <geometry><mesh filename="package://yahboomcar_description/meshes/base_link_X3.STL"/></geometry>
+      <material name="Green"/>
+    </visual>
+    <collision>
+      <origin xyz="0 0 0" rpy="0 0 0"/>
+      <geometry><mesh filename="package://yahboomcar_description/meshes/base_link_X3.STL"/></geometry>
+    </collision>
+  </link>
+  <!-- front_right_wheel -->
+  <link name="front_right_wheel">
+    <inertial>
+      <origin xyz="1.9051E-06 -2.3183E-07 -0.00064079" rpy="0 0 0"/>
+      <mass value="0.051532"/>
+      <inertia ixx="1.4595E-05" ixy="-4.3975E-10" ixz="4.415E-10"
+               iyy="1.4594E-05" iyz="-1.7476E-09" izz="2.4264E-05"/>
+    </inertial>
+    <visual>
+      <origin xyz="0 0 0" rpy="0 0 0"/>
+      <geometry><mesh filename="package://yahboomcar_description/meshes/front_right_wheel_X3.STL"/></geometry>
+      <material name="White"/>
+    </visual>
+    <collision>
+      <origin xyz="0 0 0" rpy="0 0 0"/>
+      <geometry><mesh filename="package://yahboomcar_description/meshes/front_right_wheel_X3.STL"/></geometry>
+    </collision>
+  </link>
+  <!-- front_left_wheel -->
+  <link name="front_left_wheel">
+    <inertial>
+      <origin xyz="2.3728E-06 -9.4228E-07 0.00064068" rpy="0 0 0"/>
+      <mass value="0.051543"/>
+      <inertia ixx="1.4597E-05" ixy="-4.7945E-10" ixz="-2.4786E-10"
+               iyy="1.4598E-05" iyz="1.7972E-09" izz="2.4267E-05"/>
+    </inertial>
+    <visual>
+      <origin xyz="0 0 0" rpy="0 0 0"/>
+      <geometry><mesh filename="package://yahboomcar_description/meshes/front_left_wheel_X3.STL"/></geometry>
+      <material name="White"/>
+    </visual>
+    <collision>
+      <origin xyz="0 0 0" rpy="0 0 0"/>
+      <geometry><mesh filename="package://yahboomcar_description/meshes/front_left_wheel_X3.STL"/></geometry>
+    </collision>
+  </link>
+  <!-- back_right_wheel -->
+  <link name="back_right_wheel">
+    <inertial>
+      <origin xyz="-1.75924169923403E-06 1.28388821071107E-06 -0.000590549296238266" rpy="0 0 0"/>
+      <mass value="0.051540174053366"/>
+      <inertia ixx="1.45974152250002E-05" ixy="1.94850559178397E-10" ixz="-1.61846387282284E-09"
+               iyy="1.4596501955693E-05"  iyz="-6.27904057423818E-10" izz="2.42663091380451E-05"/>
+    </inertial>
+    <visual>
+      <origin xyz="0 0 0" rpy="0 0 0"/>
+      <geometry><mesh filename="package://yahboomcar_description/meshes/back_right_wheel_X3.STL"/></geometry>
+      <material name="White"/>
+    </visual>
+    <collision>
+      <origin xyz="0 0 0" rpy="0 0 0"/>
+      <geometry><mesh filename="package://yahboomcar_description/meshes/back_right_wheel_X3.STL"/></geometry>
+    </collision>
+  </link>
+  <!-- back_left_wheel -->
+  <link name="back_left_wheel">
+    <inertial>
+      <origin xyz="-4.01213085227115E-07 2.04910264598596E-06 0.000590775697051377" rpy="0 0 0"/>
+      <mass value="0.0515309299357028"/>
+      <inertia ixx="1.45942986129926E-05" ixy="-3.19787215398093E-10" ixz="1.74943062058915E-09"
+               iyy="1.45948727598913E-05" iyz="1.61769812110049E-10"  izz="2.4263683888153E-05"/>
+    </inertial>
+    <visual>
+      <origin xyz="0 0 0" rpy="0 0 0"/>
+      <geometry><mesh filename="package://yahboomcar_description/meshes/back_left_wheel_X3.STL"/></geometry>
+      <material name="White"/>
+    </visual>
+    <collision>
+      <origin xyz="0 0 0" rpy="0 0 0"/>
+      <geometry><mesh filename="package://yahboomcar_description/meshes/back_left_wheel_X3.STL"/></geometry>
+    </collision>
+  </link>
+  <!-- laser_link -->
+  <link name="laser_link">
+    <inertial>
+      <origin xyz="-0.0176558922685589 0.000671805271544437 0.0219302095894866" rpy="0 0 0"/>
+      <mass value="0.0483909504209895"/>
+      <inertia ixx="1.58456966399128E-05" ixy="-4.23913983850005E-07" ixz="-2.09597897904374E-07"
+               iyy="3.89262522903605E-05" iyz="3.24809725932687E-07"  izz="4.86230801106223E-05"/>
+    </inertial>
+    <visual>
+      <origin xyz="0 0 0" rpy="0 0 0"/>
+      <geometry><mesh filename="package://yahboomcar_description/meshes/laser_link.STL"/></geometry>
+      <material name="White"/>
+    </visual>
+    <collision>
+      <origin xyz="0 0 0" rpy="0 0 0"/>
+      <geometry><mesh filename="package://yahboomcar_description/meshes/laser_link.STL"/></geometry>
+    </collision>
+  </link>
+  <!-- camera_link -->
+  <link name="camera_link">
+    <inertial>
+      <origin xyz="0 0 0" rpy="0 0 0"/>
+      <mass value="0"/>
+      <inertia ixx="0" ixy="0" ixz="0" iyy="0" iyz="0" izz="0"/>
+    </inertial>
+    <visual>
+      <origin xyz="0 0 0" rpy="0 0 0"/>
+      <geometry><mesh filename="package://yahboomcar_description/meshes/camera_link.STL"/></geometry>
+      <material name="White"/>
+    </visual>
+    <collision>
+      <origin xyz="0 0 0" rpy="0 0 0"/>
+      <geometry><mesh filename="package://yahboomcar_description/meshes/camera_link.STL"/></geometry>
+    </collision>
+  </link>
+  <!-- ═══════════════════════════════════════════════════════════════════════
+       JOINTS
+  ══════════════════════════════════════════════════════════════════════════ -->
+  <joint name="base_joint" type="fixed">
+    <parent link="base_footprint"/><child link="base_link"/>
+    <origin xyz="0.0 0.0 0.0815" rpy="0 0 0"/>
+  </joint>
+  <joint name="base_imu" type="fixed">
+    <parent link="base_link"/><child link="imu_link"/>
+    <origin xyz="-0.06 0.01 0.01" rpy="0 3.1415 1.5707"/>
+  </joint>
+  <!--
+      IMPORTANT : les noms de joints ci-dessous (front_left_joint, etc.)
+      DOIVENT correspondre exactement au YAML et au hardware plugin.
+      Ne pas ajouter de préfixe namespace ici.
+  -->
+  <joint name="front_right_joint" type="continuous">
+    <origin xyz="0.08 -0.0845 -0.0389" rpy="-1.5703 0 3.14159"/>
+    <parent link="base_link"/><child link="front_right_wheel"/>
+    <axis xyz="0 0 1"/>
+    <limit effort="100" velocity="10"/>
+  </joint>
+  <joint name="front_left_joint" type="continuous">
+    <origin xyz="0.08 0.084492 -0.0389" rpy="1.5703 0 0"/>
+    <parent link="base_link"/><child link="front_left_wheel"/>
+    <axis xyz="0 0 1"/>
+    <limit effort="100" velocity="10"/>
+  </joint>
+  <joint name="back_right_joint" type="continuous">
+    <origin xyz="-0.08 -0.0845 -0.03946" rpy="-1.57 0 3.14159"/>
+    <parent link="base_link"/><child link="back_right_wheel"/>
+    <axis xyz="0 0 1"/>
+    <limit effort="100" velocity="10"/>
+  </joint>
+  <joint name="back_left_joint" type="continuous">
+    <origin xyz="-0.08 0.084492 -0.03954" rpy="1.5703 0 0"/>
+    <parent link="base_link"/><child link="back_left_wheel"/>
+    <axis xyz="0 0 1"/>
+    <limit effort="100" velocity="10"/>
+  </joint>
+  <joint name="laser_joint" type="fixed">
+    <origin xyz="0.0435 5.25826986680105E-05 0.11" rpy="0 0 0"/>
+    <parent link="base_link"/><child link="laser_link"/>
+  </joint>
+  <joint name="camera_joint" type="fixed">
+    <origin xyz="0.057105 1.7948E-05 0.03755" rpy="0 0 0"/>
+    <parent link="base_link"/><child link="camera_link"/>
+  </joint>
+  <!-- ═══════════════════════════════════════════════════════════════════════
+       BLOC ros2_control  —  ÉTAIT TOTALEMENT ABSENT → BUG 1 + 2 RÉGLÉS ICI
+       Le plugin MecarosmasterHardware reçoit serial_port et car_type.
+  ══════════════════════════════════════════════════════════════════════════ -->
+  <ros2_control name="MecarosmasterSystem" type="system">
+    <hardware>
+      <plugin>mecarosmaster_ros2_control/MecarosmasterHardware</plugin>
+      <param name="serial_port">$(arg serial_port)</param>
+      <param name="car_type">$(arg car_type)</param>
+      <param name="ticks_per_rev">1625</param>
+      <param name="wheel_radius">0.045</param>
+      <param name="wheel_sep_x">0.08</param>
+      <param name="wheel_sep_y">0.0845</param>
+      <param name="cmd_delay">0.002</param>
+      <param name="cmd_deadband">0.0001</param>
+      <param name="debug">false</param>
+    </hardware>
+    <!--
+        Ordre : FL=0  FR=1  RL=2  RR=3  (identique à hw_cmd_[] dans le plugin)
+        Noms : EXACTEMENT ceux déclarés dans les joints ci-dessus.
+    -->
+    <joint name="front_left_joint">
+      <command_interface name="velocity">
+        <param name="min">-10</param>
+        <param name="max"> 10</param>
+      </command_interface>
+      <state_interface name="position"/>
+      <state_interface name="velocity"/>
+    </joint>
+    <joint name="front_right_joint">
+      <command_interface name="velocity">
+        <param name="min">-10</param>
+        <param name="max"> 10</param>
+      </command_interface>
+      <state_interface name="position"/>
+      <state_interface name="velocity"/>
+    </joint>
+    <joint name="back_left_joint">
+      <command_interface name="velocity">
+        <param name="min">-10</param>
+        <param name="max"> 10</param>
+      </command_interface>
+      <state_interface name="position"/>
+      <state_interface name="velocity"/>
+    </joint>
+    <joint name="back_right_joint">
+      <command_interface name="velocity">
+        <param name="min">-10</param>
+        <param name="max"> 10</param>
+      </command_interface>
+      <state_interface name="position"/>
+      <state_interface name="velocity"/>
+    </joint>
+  </ros2_control>
 </robot>
